File: kicad/NurseQuacky.kicad_sch (KiCad schematic)
At the start: 31 parts, among them J1 Barrel_Jack_Switch, Q1 2N3904, U1 TL072

Commit message: Small fixes for rev01 schematic.
Parts:
- removed J1: Barrel_Jack_Switch, symbol Connector:Barrel_Jack_Switch
- added C11: 100uF, Capacitor_THT:CP_Radial_D5.0mm_P2.00mm, symbol Device:C_Polarized_US
- added C3: .0047uF, Capacitor_THT:C_Rect_L7.2mm_W2.5mm_P5.00mm_FKS2_FKP2_MKS2_MKP2, symbol Device:C
- added D1: 1N5817, Diode_THT:D_DO-41_SOD81_P7.62mm_Horizontal, symbol Device:D_Schottky
- added J1: A_08-LC-TT, digikey-footprints:SOCKET_DIP-8_7.62mm_Conn, symbol dk_Sockets-for-ICs-Transistors:A_08-LC-TT
- added R16, R4: 1M, Resistor_THT:R_Axial_DIN0207_L6.3mm_D2.5mm_P7.62mm_Horizontal, symbol Device:R_US
- ATK1: renamed from ATTACK; footprint (none) -> PedalBuilding:Alpha_16mm_RightAngle; Sourcing (none) -> https://www.taydaelectronics.com/p1-b1k-ohm-linear-taper-po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
- C1: renamed from C8; footprint (none) -> Capacitor_THT:CP_Radial_D5.0mm_P2.00mm; Sourcing (none) -> https://www.taydaelectronics.com/100uf-16v-105c-aluminum-ra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
- C10: renamed from C7; footprint (none) -> Capacitor_THT:C_Rect_L7.2mm_W2.5mm_P5.00mm_FKS2_FKP2_MKS2_MKP2; Sourcing (none) -> https://www.taydaelectronics.com/wima-mks2-0-1uf-63v-10-pol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
- C2: renamed from C9; footprint (none) -> Capacitor_THT:CP_Radial_D5.0mm_P2.00mm; Sourcing (none) -> https://www.taydaelectronics.com/47uf-25v-105c-aluminum-rad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
- C4: renamed from C1; footprint (none) -> Capacitor_THT:C_Rect_L7.2mm_W2.5mm_P5.00mm_FKS2_FKP2_MKS2_MKP2; Sourcing (none) -> https://www.taydaelectronics.com/wima-10nf-0-01uf-100v-5-po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
- C5: renamed from C2; footprint (none) -> Capacitor_THT:C_Rect_L7.2mm_W2.5mm_P5.00mm_FKS2_FKP2_MKS2_MKP2; Sourcing (none) -> https://www.taydaelectronics.com/wima-10nf-0-01uf-100v-5-po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
- C6: renamed from C5; footprint (none) -> Capacitor_THT:C_Rect_L7.2mm_W2.5mm_P5.00mm_FKS2_FKP2_MKS2_MKP2; Sourcing (none) -> https://www.taydaelectronics.com/wima-fks2-4-7-nf-0-0047uf-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
- C7: renamed from C4; footprint (none) -> Capacitor_THT:C_Rect_L7.2mm_W2.5mm_P5.00mm_FKS2_FKP2_MKS2_MKP2; Sourcing (none) -> https://www.taydaelectronics.com/wima-fks2-4-7-nf-0-0047uf-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
- C8: renamed from C6; footprint (none) -> Capacitor_THT:C_Rect_L7.2mm_W2.5mm_P5.00mm_FKS2_FKP2_MKS2_MKP2; Sourcing (none) -> https://www.taydaelectronics.com/wima-fks2-100nf-0-001uf-10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
- C9: renamed from C3; footprint (none) -> Capacitor_THT:CP_Radial_D5.0mm_P2.00mm; Sourcing (none) -> https://www.taydaelectronics.com/22uf-25v-85c-radial-electr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
- D2: renamed from D1; footprint (none) -> digikey-footprints:LED_3mm_Radial; Sourcing (none) -> https://www.taydaelectronics.com/led-3mm-red.html
- D3: renamed from D2; footprint (none) -> digikey-footprints:LED_3mm_Radial; Sourcing (none) -> https://www.taydaelectronics.com/led-3mm-red.html
- Q1: Sourcing (none) -> https://www.taydaelectronics.com/2n3904-npn-general-propose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
- R1: renamed from R13; footprint (none) -> Resistor_THT:R_Axial_DIN0207_L6.3mm_D2.5mm_P7.62mm_Horizontal; Sourcing (none) -> https://www.taydaelectronics.com/resistors/1-4w-metal-film-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
- R10: renamed from R5; footprint (none) -> Resistor_THT:R_Axial_DIN0207_L6.3mm_D2.5mm_P7.62mm_Horizontal; Sourcing (none) -> https://www.taydaelectronics.com/resistors/1-4w-metal-film-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
- R11: renamed from R7; footprint (none) -> Resistor_THT:R_Axial_DIN0207_L6.3mm_D2.5mm_P7.62mm_Horizontal; Sourcing (none) -> https://www.taydaelectronics.com/resistors/1-4w-metal-film-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
- R12: renamed from R3; footprint (none) -> Resistor_THT:R_Axial_DIN0207_L6.3mm_D2.5mm_P7.62mm_Horizontal; Sourcing (none) -> https://www.taydaelectronics.com/resistors/1-4w-metal-film-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
- R13: renamed from R11; footprint (none) -> Resistor_THT:R_Axial_DIN0207_L6.3mm_D2.5mm_P7.62mm_Horizontal; Sourcing (none) -> https://www.taydaelectronics.com/resistors/1-4w-metal-film-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
- R14: renamed from R8; footprint (none) -> Resistor_THT:R_Axial_DIN0207_L6.3mm_D2.5mm_P7.62mm_Horizontal; Sourcing (none) -> https://www.taydaelectronics.com/resistors/1-4w-metal-film-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
- R15: renamed from R9; footprint (none) -> Resistor_THT:R_Axial_DIN0207_L6.3mm_D2.5mm_P7.62mm_Horizontal; Sourcing (none) -> https://www.taydaelectronics.com/resistors/1-4w-metal-film-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
- R2: renamed from R14; footprint (none) -> Resistor_THT:R_Axial_DIN0207_L6.3mm_D2.5mm_P7.62mm_Horizontal; Sourcing (none) -> https://www.taydaelectronics.com/resistors/1-4w-metal-film-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
- R3: renamed from R12; footprint (none) -> Resistor_THT:R_Axial_DIN0207_L6.3mm_D2.5mm_P7.62mm_Horizontal; Sourcing (none) -> https://www.taydaelectronics.com/resistors/1-4w-metal-film-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
- R5: renamed from R1; footprint (none) -> Resistor_THT:R_Axial_DIN0207_L6.3mm_D2.5mm_P7.62mm_Horizontal; Sourcing (none) -> https://www.taydaelectronics.com/resistors/1-4w-metal-film-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
- R6: renamed from R4; footprint (none) -> Resistor_THT:R_Axial_DIN0207_L6.3mm_D2.5mm_P7.62mm_Horizontal; Sourcing (none) -> https://www.taydaelectronics.com/resistors/1-4w-metal-film-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
- R7: renamed from R6; footprint (none) -> Resistor_THT:R_Axial_DIN0207_L6.3mm_D2.5mm_P7.62mm_Horizontal; Sourcing (none) -> https://www.taydaelectronics.com/resistors/1-4w-metal-film-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
- R8: renamed from R10; footprint (none) -> Resistor_THT:R_Axial_DIN0207_L6.3mm_D2.5mm_P7.62mm_Horizontal; Sourcing (none) -> https://www.taydaelectronics.com/resistors/1-4w-metal-film-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
- R9: renamed from R2; footprint (none) -> Resistor_THT:R_Axial_DIN0207_L6.3mm_D2.5mm_P7.62mm_Horizontal; Sourcing (none) -> https://www.taydaelectronics.com/resistors/1-4w-metal-film-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
- RNG1: renamed from RANGE; footprint (none) -> PedalBuilding:Alpha_16mm_RightAngle; Sourcing (none) -> https://www.taydaelectronics.com/p1-b25k-ohm-linear-taper-p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
- SENS1: renamed from SENS; footprint (none) -> PedalBuilding:Alpha_16mm_RightAngle; Sourcing (none) -> https://www.taydaelectronics.com/b100k-ohm-linear-taper-pot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
- U1: footprint (none) -> digikey-footprints:DIP-8_W7.62mm; Sourcing (none) -> https://www.taydaelectronics.com/tl072-low-noise-j-fet-dual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
Connections:
- net Earth: now also R16.1, R4.2
- net INPUT: now also C3.1; no longer C4.1, R5.1, SENS1.1
- net OUTPUT: now also C11.2, R16.2; no longer C10.1, R13.2
- net at C1.1, R1.1, R3.2: now also D1.1 (K)
- new net: C3.2, C4.1, R4.1, R5.1, SENS1.1
- new net: C10.1, C11.1, R13.2
- new net VCC: D1.2 (A)
- no-connect marks 0 -> 8
Other:
- company: Author: Noah Iniguez, https://github.com/noahssarcastic -> (none)
- moved on the sheet: ATK1, C1, C10, C2, C4, C5, C6, C7, C8, C9, D2, D3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
